Commit message: fix: fix multiple issues
- Fix executable name for amir_ros compatibility
- Resolve self-collision problem
- Add launch arguments to exclude rover
- Group and rename RViz config file

File: r4_description/urdf/robovie_r4_rover.xacro (robot description, xacro)
@@ -1,8 +1,9 @@
 <?xml version="1.0" ?>
 <robot name="robovie_r4" xmlns:xacro="http://www.ros.org/wiki/xacro">
-<xacro:include filename="$(find r4_description)/urdf/materials.xacro" />
+<!-- <xacro:include filename="$(find r4_description)/urdf/materials.xacro" /> -->
+<xacro:include filename="$(find megarover_description)/urdf/mega3_base_model.xacro" />
+<xacro:include filename="$(find r4_description)/urdf/robovie_r4_base.xacro" />
 <!-- <xacro:include filename="$(find r4_description)/urdf/robovie_r4.trans" /> -->
 <!-- <xacro:include filename="$(find r4_description)/urdf/robovie_r4.gazebo" /> -->
-<xacro:include filename="$(find megarover_description)/urdf/mega3_base_model.xacro" />
 <joint name="rover_joint" type="fixed">
   <origin xyz="0.0 0.0 0.015" rpy="0 0 0"/>
@@ -10,353 +11,3 @@
   <child link="torso_link_r4"/>
 </joint>
-<link name="tcp_left">
-  <visual>
-    <geometry>
-      <box size="0.01 0.01 0.01"/>
-    </geometry>
-    <material name="red">
-      <color rgba="1.0 0.0 0.0 0.6"/>
-    </material>
-  </visual>
-</link>
-<joint name="tcp_left_joint" type="fixed">
-   <!-- X軸の正方向が前 -->
-  <origin xyz="${-0.032-0.003262} ${-0.0375+0.037358} ${-0.168+0.000071}" rpy="0 0 0"/>
-  <parent link="l_hand_1"/>
-  <child link="tcp_left"/>
-</joint>
-<link name="tcp_right">
-  <visual>
-    <geometry>
-      <box size="0.01 0.01 0.01"/>
-    </geometry>
-    <material name="red">
-      <color rgba="1.0 0.0 0.0 0.6"/>
-    </material>
-  </visual>
-</link>
-<joint name="tcp_right_joint" type="fixed">
-   <!-- X軸の正方向が前 -->
-  <origin xyz="${0.032-0.003262} ${-0.0375+0.037358} ${-0.168+0.000071}" rpy="0 0 0"/>
-  <parent link="r_hand_1"/>
-  <child link="tcp_right"/>
-</joint>
-<link name="torso_link_r4">
-  <inertial>
-    <origin xyz="0.000614628156240865 0.001148796640096465 0.4251467803392016" rpy="0 0 0"/>
-    <mass value="26.157484443567014"/>
-    <inertia ixx="2.07336" iyy="2.086701" izz="0.73142" ixy="0.001276" iyz="-0.012697" ixz="-0.003299"/>
-  </inertial>
-  <visual>
-    <origin xyz="0 0 0" rpy="0 0 0"/>
-    <geometry>
-      <mesh filename="package://r4_description/meshes/torso_link_r4.stl" scale="0.001 0.001 0.001"/>
-    </geometry>
-    <material name="silver-r4"/>
-  </visual>
-  <collision>
-    <origin xyz="0 0 0" rpy="0 0 0"/>
-    <geometry>
-      <mesh filename="package://r4_description/meshes/torso_link_r4.stl" scale="0.001 0.001 0.001"/>
-    </geometry>
-  </collision>
-</link>
-<link name="l_shoulder_1">
-  <inertial>
-    <origin xyz="-0.037852630361978945 0.00325917485373633 0.0033240289687475055" rpy="0 0 0"/>
-    <mass value="1.3261389056969144"/>
-    <inertia ixx="0.001184" iyy="0.002087" izz="0.0021" ixy="7.9e-05" iyz="-7e-06" ixz="8.1e-05"/>
-  </inertial>
-  <visual>
-    <origin xyz="0.134657 -0.011781 -0.696078" rpy="0 0 0"/>
-    <geometry>
-      <mesh filename="package://r4_description/meshes/l_shoulder_1.stl" scale="0.001 0.001 0.001"/>
-    </geometry>
-    <material name="silver-r4"/>
-  </visual>
-  <collision>
-    <origin xyz="0.134657 -0.011781 -0.696078" rpy="0 0 0"/>
-    <geometry>
-      <mesh filename="package://r4_description/meshes/l_shoulder_1.stl" scale="0.001 0.001 0.001"/>
-    </geometry>
-  </collision>
-</link>
-<link name="r_shoulder_1">
-  <inertial>
-    <origin xyz="0.03784353770491708 0.0033633036532929993 0.0033238304731996182" rpy="0 0 0"/>
-    <mass value="1.3261389056969144"/>
-    <inertia ixx="0.001184" iyy="0.002087" izz="0.0021" ixy="-8e-05" iyz="-7e-06" ixz="-8.1e-05"/>
-  </inertial>
-  <visual>
-    <origin xyz="-0.134657 -0.011781 -0.696078" rpy="0 0 0"/>
-    <geometry>
-      <mesh filename="package://r4_description/meshes/r_shoulder_1.stl" scale="0.001 0.001 0.001"/>
-    </geometry>
-    <material name="silver-r4"/>
-  </visual>
-  <collision>
-    <origin xyz="-0.134657 -0.011781 -0.696078" rpy="0 0 0"/>
-    <geometry>
-      <mesh filename="package://r4_description/meshes/r_shoulder_1.stl" scale="0.001 0.001 0.001"/>
-    </geometry>
-  </collision>
-</link>
-<link name="neck_yaw_link_1">
-  <inertial>
-    <origin xyz="-0.001909747489438639 0.002260196795276822 0.016471266556445152" rpy="0 0 0"/>
-    <mass value="0.14692716936201883"/>
-    <inertia ixx="0.000101" iyy="5.2e-05" izz="8.9e-05" ixy="-0.0" iyz="0.0" ixz="0.0"/>
-  </inertial>
-  <visual>
-    <origin xyz="-0.0 -0.0 -0.823" rpy="0 0 0"/>
-    <geometry>
-      <mesh filename="package://r4_description/meshes/neck_yaw_link_1.stl" scale="0.001 0.001 0.001"/>
-    </geometry>
-    <material name="silver-r4"/>
-  </visual>
-  <collision>
-    <origin xyz="-0.0 -0.0 -0.823" rpy="0 0 0"/>
-    <geometry>
-      <mesh filename="package://r4_description/meshes/neck_yaw_link_1.stl" scale="0.001 0.001 0.001"/>
-    </geometry>
-  </collision>
-</link>
-<link name="neck_roll_link_1">
-  <inertial>
-    <origin xyz="0.0005064508038095865 -0.0221821481261072 0.01791091802139455" rpy="0 0 0"/>
-    <mass value="1.1480815935567241"/>
-    <inertia ixx="0.000617" iyy="0.000684" izz="0.000457" ixy="-0.0" iyz="1e-06" ixz="0.0"/>
-  </inertial>
-  <visual>
-    <origin xyz="0.0 -0.0245 -0.85" rpy="0 0 0"/>
-    <geometry>
-      <mesh filename="package://r4_description/meshes/neck_roll_link_1.stl" scale="0.001 0.001 0.001"/>
-    </geometry>
-    <material name="silver-r4"/>
-  </visual>
-  <collision>
-    <origin xyz="0.0 -0.0245 -0.85" rpy="0 0 0"/>
-    <geometry>
-      <mesh filename="package://r4_description/meshes/neck_roll_link_1.stl" scale="0.001 0.001 0.001"/>
-    </geometry>
-  </collision>
-</link>
-<link name="head_1">
-  <inertial>
-    <origin xyz="-0.026505019942840876 -0.0016225754455137511 0.09761714285669354" rpy="0 0 0"/>
-    <mass value="7.576311537618501"/>
-    <inertia ixx="0.051342" iyy="0.073001" izz="0.076119" ixy="4e-06" iyz="0.00224" ixz="-7e-06"/>
-  </inertial>
-  <visual>
-    <origin xyz="-0.0265 -0.0 -0.85" rpy="0 0 0"/>
-    <geometry>
-      <mesh filename="package://r4_description/meshes/head_1.stl" scale="0.001 0.001 0.001"/>
-    </geometry>
-    <material name="silver-r4"/>
-  </visual>
-  <collision>
-    <origin xyz="-0.0265 -0.0 -0.85" rpy="0 0 0"/>
-    <geometry>
-      <mesh filename="package://r4_description/meshes/head_1.stl" scale="0.001 0.001 0.001"/>
-    </geometry>
-  </collision>
-</link>
-<link name="l_arm_1">
-  <inertial>
-    <origin xyz="-0.01171737181229937 -0.029404568328405267 -0.05915031814076621" rpy="0 0 0"/>
-    <mass value="0.7243594855307846"/>
-    <inertia ixx="0.002358" iyy="0.001919" izz="0.001152" ixy="-3.9e-05" iyz="1.3e-05" ixz="-0.00016"/>
-  </inertial>
-  <visual>
-    <origin xyz="0.182292 -0.015949 -0.700261" rpy="0 0 0"/>
-    <geometry>
-      <mesh filename="package://r4_description/meshes/l_arm_1.stl" scale="0.001 0.001 0.001"/>
-    </geometry>
-    <material name="silver-r4"/>
-  </visual>
-  <collision>
-    <origin xyz="0.182292 -0.015949 -0.700261" rpy="0 0 0"/>
-    <geometry>
-      <mesh filename="package://r4_description/meshes/l_arm_1.stl" scale="0.001 0.001 0.001"/>
-    </geometry>
-  </collision>
-</link>
-<link name="r_arm_1">
-  <inertial>
-    <origin xyz="0.011717377079669272 -0.0294046286501487 -0.059150318025778414" rpy="0 0 0"/>
-    <mass value="0.7243594855307846"/>
-    <inertia ixx="0.002358" iyy="0.001919" izz="0.001152" ixy="3.9e-05" iyz="1.3e-05" ixz="0.00016"/>
-  </inertial>
-  <visual>
-    <origin xyz="-0.182292 -0.015949 -0.700261" rpy="0 0 0"/>
-    <geometry>
-      <mesh filename="package://r4_description/meshes/r_arm_1.stl" scale="0.001 0.001 0.001"/>
-    </geometry>
-    <material name="silver-r4"/>
-  </visual>
-  <collision>
-    <origin xyz="-0.182292 -0.015949 -0.700261" rpy="0 0 0"/>
-    <geometry>
-      <mesh filename="package://r4_description/meshes/r_arm_1.stl" scale="0.001 0.001 0.001"/>
-    </geometry>
-  </collision>
-</link>
-<link name="l_elbow_1">
-  <inertial>
-    <origin xyz="0.013707025391952676 -0.0012488485865315528 -0.02739437843448611" rpy="0 0 0"/>
-    <mass value="1.3817415156964064"/>
-    <inertia ixx="0.000976" iyy="0.000677" izz="0.001046" ixy="-2.6e-05" iyz="-8e-06" ixz="0.000103"/>
-  </inertial>
-  <visual>
-    <origin xyz="0.192122 -0.016592 -0.587692" rpy="0 0 0"/>
-    <geometry>
-      <mesh filename="package://r4_description/meshes/l_elbow_1.stl" scale="0.001 0.001 0.001"/>
-    </geometry>
-    <material name="silver-r4"/>
-  </visual>
-  <collision>
-    <origin xyz="0.192122 -0.016592 -0.587692" rpy="0 0 0"/>
-    <geometry>
-      <mesh filename="package://r4_description/meshes/l_elbow_1.stl" scale="0.001 0.001 0.001"/>
-    </geometry>
-  </collision>
-</link>
-<link name="r_elbow_1">
-  <inertial>
-    <origin xyz="-0.01370702179735625 -0.001248889751733982 -0.027394378356015325" rpy="0 0 0"/>
-    <mass value="1.3817415156964064"/>
-    <inertia ixx="0.000976" iyy="0.000677" izz="0.001046" ixy="2.6e-05" iyz="-8e-06" ixz="-0.000103"/>
-  </inertial>
-  <visual>
-    <origin xyz="-0.192122 -0.016592 -0.587692" rpy="0 0 0"/>
-    <geometry>
-      <mesh filename="package://r4_description/meshes/r_elbow_1.stl" scale="0.001 0.001 0.001"/>
-    </geometry>
-    <material name="silver-r4"/>
-  </visual>
-  <collision>
-    <origin xyz="-0.192122 -0.016592 -0.587692" rpy="0 0 0"/>
-    <geometry>
-      <mesh filename="package://r4_description/meshes/r_elbow_1.stl" scale="0.001 0.001 0.001"/>
-    </geometry>
-  </collision>
-</link>
-<link name="l_hand_1">
-  <inertial>
-    <origin xyz="-0.03076625385048895 -0.03513212246685853 -0.09224704680541085" rpy="0 0 0"/>
-    <mass value="1.3532058766017583"/>
-    <inertia ixx="0.005572" iyy="0.005107" izz="0.002078" ixy="-4.2e-05" iyz="3.8e-05" ixz="-0.000499"/>
-  </inertial>
-  <visual>
-    <origin xyz="0.174797 -0.015021 -0.557059" rpy="0 0 0"/>
-    <geometry>
-      <mesh filename="package://r4_description/meshes/l_hand_1.stl" scale="0.001 0.001 0.001"/>
-    </geometry>
-    <material name="silver-r4"/>
-  </visual>
-  <collision>
-    <origin xyz="0.174797 -0.015021 -0.557059" rpy="0 0 0"/>
-    <geometry>
-      <mesh filename="package://r4_description/meshes/l_hand_1.stl" scale="0.001 0.001 0.001"/>
-    </geometry>
-  </collision>
-</link>
-<link name="r_hand_1">
-  <inertial>
-    <origin xyz="0.030766274993907133 -0.03513236460057082 -0.09224704634384401" rpy="0 0 0"/>
-    <mass value="1.3532058766017574"/>
-    <inertia ixx="0.005572" iyy="0.005107" izz="0.002078" ixy="4.2e-05" iyz="3.8e-05" ixz="0.000499"/>
-  </inertial>
-  <visual>
-    <origin xyz="-0.174797 -0.015021 -0.557059" rpy="0 0 0"/>
-    <geometry>
-      <mesh filename="package://r4_description/meshes/r_hand_1.stl" scale="0.001 0.001 0.001"/>
-    </geometry>
-    <material name="silver-r4"/>
-  </visual>
-  <collision>
-    <origin xyz="-0.174797 -0.015021 -0.557059" rpy="0 0 0"/>
-    <geometry>
-      <mesh filename="package://r4_description/meshes/r_hand_1.stl" scale="0.001 0.001 0.001"/>
-    </geometry>
-  </collision>
-</link>
-<!-- joints *****************************************-->
-<joint name="l_shoulder_pitch" type="revolute">
-  <origin xyz="-0.134657 0.011781 0.696078" rpy="0 0 0"/>
-  <parent link="torso_link_r4"/>
-  <child link="l_shoulder_1"/>
-  <axis xyz="-0.992404 0.086824 0.087156"/>
-  <limit upper="${70*pi/180}" lower="${-250*pi/180}" effort="100" velocity="100"/>
-</joint>
-<joint name="l_shoulder_roll" type="revolute">
-  <origin xyz="${-0.045008-0.002627} ${0.034253-0.030085} ${0.004126+0.000057}" rpy="0 0 0"/>
-  <parent link="l_shoulder_1"/>
-  <child link="l_arm_1"/>
-  <axis xyz="0.08699 0.996207 -0.001899"/>
-  <limit upper="${170*pi/180}" lower="${-10*pi/180}" effort="100" velocity="100"/>
-</joint>
-<joint name="l_elbow_yaw" type="revolute">
-  <origin xyz="${-0.012457+0.002627} ${-0.029442+0.030085} ${-0.112512-0.000057}" rpy="0 0 0"/>
-  <parent link="l_arm_1"/>
-  <child link="l_elbow_1"/>
-  <axis xyz="-0.08699 0.005697 -0.996193"/>
-  <limit upper="${pi/2}" lower="${-pi/2}" effort="100" velocity="100"/>
-</joint>
-<joint name="l_elbow_bend" type="revolute">
-  <origin xyz="${0.020587-0.003262} ${0.035787-0.037358} ${-0.030704-0.000071}" rpy="0 0 0"/>
-  <parent link="l_elbow_1"/>
-  <child link="l_hand_1"/>
-  <axis xyz="0.08699 0.996207 -0.001899"/>
-  <limit upper="${5*pi/180}" lower="${-125*pi/180}" effort="100" velocity="100"/>
-</joint>
-<joint name="r_shoulder_pitch" type="revolute">
-  <origin xyz="0.134657 0.011781 0.696078" rpy="0 0 0"/>
-  <parent link="torso_link_r4"/>
-  <child link="r_shoulder_1"/>
-  <axis xyz="0.992404 0.086824 0.087156"/>
-  <limit upper="${250*pi/180}" lower="${-70*pi/180}" effort="100" velocity="100"/>
-</joint>
-<joint name="r_shoulder_roll" type="revolute">
-  <origin xyz="${0.045008+0.002627} ${0.034253-0.030085} ${0.004126+0.000057}" rpy="0 0 0"/>
-  <parent link="r_shoulder_1"/>
-  <child link="r_arm_1"/>
-  <axis xyz="-0.08699 0.996207 -0.001899"/>
-  <limit lower="${-170*pi/180}" upper="${10*pi/180}" effort="100" velocity="100"/>
-</joint>
-<joint name="r_elbow_yaw" type="revolute">
-  <origin xyz="${0.012457-0.002627} ${-0.029442+0.030085} ${-0.112512-0.000057}" rpy="0 0 0"/>
-  <parent link="r_arm_1"/>
-  <child link="r_elbow_1"/>
-  <axis xyz="0.08699 0.005697 -0.996193"/>
-  <limit upper="${pi/2}" lower="${-pi/2}" effort="100" velocity="100"/>
-</joint>
-<joint name="r_elbow_bend" type="revolute">
-  <origin xyz="${-0.020587+0.003262} ${0.035787-0.037358} ${-0.030704-0.000071}" rpy="0 0 0"/>
-  <parent link="r_elbow_1"/>
-  <child link="r_hand_1"/>
-  <axis xyz="-0.08699 0.996207 -0.001899"/>
-  <limit upper="${125*pi/180}" lower="${-5*pi/180}" effort="100" velocity="100"/>
-</joint>
-<joint name="neck_yaw" type="revolute">
-  <origin xyz="0.0 0.0 0.823" rpy="0 0 0"/>
-  <parent link="torso_link_r4"/>
-  <child link="neck_yaw_link_1"/>
-  <axis xyz="0.0 0.0 1.0"/>
-  <limit upper="${pi/2}" lower="${-pi/2}" effort="100" velocity="100"/>
-</joint>
-<joint name="neck_roll" type="revolute">
-  <origin xyz="-0.0 0.0245 0.027" rpy="0 0 0"/>
-  <parent link="neck_yaw_link_1"/>
-  <child link="neck_roll_link_1"/>
-  <axis xyz="-0.0 1.0 0.0"/>
-  <limit upper="${15*pi/180}" lower="${-15*pi/180}" effort="100" velocity="100"/>
-</joint>
-<joint name="neck_pitch" type="revolute">
-  <origin xyz="0.0265 -0.0245 0.0" rpy="0 0 0"/>
-  <parent link="neck_roll_link_1"/>
-  <child link="head_1"/>
-  <axis xyz="-1.0 0.0 0.0"/>
-  <limit upper="${15*pi/180}" lower="${-30*pi/180}" effort="100" velocity="100"/>
-</joint>
 </robot>
